File: GTIA Fix.kicad_pcb (KiCad board)
At the start: 2 copper layers, 53.3 x 23.3 mm, 11 parts, among them J1 GTIA, J2 GTIA, J3 GTIA Fix, J4 GTIA Fix, U1 74LS175, U2 74HC14

Commit message: modification
Parts:
- moved J3 1.00 mm to (162.6, 129.7)
- moved J4 1.00 mm to (162.6, 114.5)
Routing:
- net GND: track 29.9 -> 8.21 mm, vias 30 -> 26
- net OSC: track 32.0 -> 28.4 mm
- net AN0_GTIA: track 8.58 -> 9.88 mm
- net +5V: track 43.6 -> 42.4 mm
- net AN2_GTIA: track 11.9 -> 13.0 mm
- net 9: track 3.66 -> 2.66 mm
- net 8: track 3.66 -> 2.66 mm
- net 7: track 3.66 -> 2.66 mm
- net 6: track 3.66 -> 2.66 mm
- net 5: track 3.66 -> 2.66 mm
- net 4: track 3.66 -> 2.66 mm
- net 2: track 3.66 -> 2.66 mm
- net 17: track 3.66 -> 2.66 mm
- net 16: track 3.66 -> 2.66 mm
- net 15: track 3.66 -> 2.66 mm
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Other:
- board size 53.3 x 23.3 mm -> 53.3 x 21.8 mm
- board text added: "1"
- board text added: "20"
- board text added: "21"
- board text added: "40"
